File: pcb/pcb.kicad_pcb (KiCad board)
At the start: 4 copper layers, 76.1 x 25.4 mm, 36 parts, among them J1 Conn_01x02_Pin, J2 Conn_01x08_Pin, J3 Conn_01x02_Pin, J4 Conn_01x02_Pin, SW1 SW_SPDT, SW2 SW_Push, U1 ATtiny85-20P, U2 FS8205A, U3 TP4056, U4 DW01A, U5 AMS1117-5.0

Commit message: production
Other:
- board text added: "Light up your camp!"
- board text added: "Mroww meow :3"
Changed lines of the file:
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@@
 		(layer "Edge.Cuts")
+	)
+	(gr_text "Light up\nyour\ncamp!"
+		(at 146.816668 54.61 -0)
+		(layer "B.SilkS")
+		(effects
+			(font
+				(size 2 2)
+				(thickness 0.4)
+				(bold yes)
+			)
+			(justify left bottom mirror)
+		)
+	)
+	(gr_text "Mroww\nmeow :3"
+		(at 112.526668 51.435 -0)
+		(layer "B.SilkS")
+		(effects
+			(font
+				(size 2 2)
+				(thickness 0.4)
+				(bold yes)
+			)
+			(justify left bottom mirror)
+		)
 	)
 	(gr_text "GND"
